File: 00-docentes/sesion-07b/udpudu/udpudu.kicad_pcb (KiCad board)
At the start: 2 copper layers, 85 x 55 mm, 20 parts, among them J1 CAIMAN, J2 TBLOCK_2, J3 CAIMAN, SW1 SW_SPDT

Commit message: editado udpudu-clase
Parts:
- added REF**: OnOff, LOGOS:OnOff, F.Cu at (82.4, 58.4)
- moved D2 2.66 mm to (130.0, 69.5)
Routing:
- net Net-(D2-A): track 9.75 -> 11.8 mm
Other:
- board text added: "@teee.udp | @lid.udp"
- board text added: "M3"
- board text removed: "SPK"
